File: hardware/eagle/flync_node.brd (EAGLE design)
At the start: 29.5 x 29.5 mm, 40 parts, among them IC1 BQ25505, IC4 TS5A23166DCUR, IC5 TLV521DCKT, IC6 TLV7031DBVR, IC7 BMD-340-A-R, T1 SI2374DSSOT23-VSHAY

Commit message: hardware: added schematic and layout as pdf
Parts:
- R7: value 1k -> 300R
Changed lines of the file:
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@@
 <attribute name="VALUE" x="5.2283" y="22.5806" size="1.27" layer="27" rot="R270" align="top-center"/>
 </element>
-<element name="R7" library="flicker-sync" package="RESC1608X55" package3d_urn="urn:adsk.eagle:package:4930386/1" value="1k" x="1.651" y="21.209" smashed="yes">
+<element name="R7" library="flicker-sync" package="RESC1608X55" package3d_urn="urn:adsk.eagle:package:4930386/1" value="300R" x="1.651" y="21.209" smashed="yes">
 <attribute name="NAME" x="1.651" y="19.4605" size="0.762" layer="25" font="vector" ratio="17" align="bottom-center"/>
 <attribute name="VALUE" x="1.651" y="19.7825" size="1.27" layer="27" align="top-center"/>
