File: hardware/eagle/flync_node.sch (EAGLE design)
At the start: 40 parts, among them IC1 BQ25505, IC4 TS5A23166DCUR, IC5 TLV521DCKT, IC6 TLV7031DBVR, IC7 BMD-340-A-R, T1 SI2374DSSOT23-VSHAY

Commit message: hardware: added schematic and layout as pdf
Parts:
- R7: value 1k -> 300R
Changed lines of the file:
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@@
 <part name="R5" library="flicker-sync" deviceset="R_SMD" device="0402" package3d_urn="urn:adsk.eagle:package:4924763/1" value="715k"/>
 <part name="R6" library="flicker-sync" deviceset="R_SMD" device="0402" package3d_urn="urn:adsk.eagle:package:4924763/1" value="1.6M"/>
-<part name="R7" library="flicker-sync" deviceset="R_SMD" device="0603" package3d_urn="urn:adsk.eagle:package:4930386/1" value="1k"/>
+<part name="R7" library="flicker-sync" deviceset="R_SMD" device="0603" package3d_urn="urn:adsk.eagle:package:4930386/1" value="300R"/>
 <part name="GND15" library="supply1" library_urn="urn:adsk.eagle:library:371" deviceset="GND" device=""/>
 <part name="H2" library="flicker-sync" deviceset="IXYSKXOB25-05X3F" device=""/>
